File: Unified Control Board/Unified Control Board.kicad_pcb (KiCad board)
At the start: 2 copper layers, 6.5 x 0.7 mm, 171 parts, among them CN1 B2B-PH-K-S(LF)(SN), CN10 B2B-PH-K-S(LF)(SN), CN11 B4B-PH-K-S(LF)(SN), CN12 B4B-PH-K-S(LF)(SN), CN201 B3B-XH-2(LF)(SN), CN202 B3B-XH-2(LF)(SN), CN203 B3B-XH-2(LF)(SN), CN3 B2B-PH-K-S(LF)(SN), CN4 B2B-PH-K-S(LF)(SN), CN5 B4B-PH-K-S(LF)(SN), CN9 B4B-PH-K-S(LF)(SN), SW1 DTSL-61N-V-T/R, SW201 TSA002A3512A02, SW202 TSA002A3512A02, U1 XT60PB-M.G.Y, U10 ESP32-S3-WROOM-1, U16 LM2596R-3.3, U2 DRV8876PWPR, U201 2.4GHz, U202 MP6541A, U203 MP6541A, U204 MP2459GJ-Z, U3 DRV8876PWPR, U5 DRV8876PWPR, U6 DRV8876PWPR, U7 TCA9546A, U9 ZDSD01GLGEAG

Commit message: Merging nets and voltage regulators
Parts:
- removed C223: 10uF/50V, ProPrj_Dri-easyedapro:C0805
- removed C224: 100nF/50V, ProPrj_Dri-easyedapro:C0603
- removed the D1 at (487.3, 144.8)
- removed D201, D203: SS36, Diode_SMD:D_SMA
- removed D5: RB050L-60TE25, MaslowMerged:SMA_L4.3-W2.7-LS5.1-RD
- removed H1: 210S-2*5P L=11.6MMGold-plated black, MaslowMerged:HDR-TH_10P-P2.54-V-M-R2-C5-S2.54
- removed H201: B-2100N10P-B110, ProPrj_Dri-easyedapro:HDR-SMD_10P-P2.54-V-M-R2-C5-S2.54-LS7.3
- removed L201: 47uH, Inductor_SMD:L_Bourns_SRN6045TA
- removed the R15 at (484.2, 144.8)
- removed R215: 124kΩ, ProPrj_Dri-easyedapro:R0402
- removed R216: 40.2kΩ, ProPrj_Dri-easyedapro:R0402
- removed R217: 100kΩ, ProPrj_Dri-easyedapro:R0402
- removed U16: LM2596R-3.3, MaslowMerged:TO-263-5_L10.2-W8.6-P1.70-LS14.4-TL
- removed U204: MP2459GJ-Z, Package_TO_SOT_SMD:SOT-23-6
- added C28: 680uF, MaslowMerged:CAP-SMD_BD10.0-L10.3-W10.3-LS10.9-FD, F.Cu at (17.7, -100.0)
- added C29: 3.3nF, ProPrj_Dri-easyedapro:C0402, F.Cu at (-109.8, 49.9)
- added C30: 68pF, ProPrj_Dri-easyedapro:C0402, F.Cu at (-109.8, 52.0)
- added C31: 100nF, ProPrj_Dri-easyedapro:C0603, F.Cu at (-109.8, 54.2)
- added C32: 10uF, ProPrj_Dri-easyedapro:C0805, F.Cu at (-105.6, 50.3)
- added C33: 22uF, ProPrj_Dri-easyedapro:C0805, F.Cu at (-105.6, 53.2)
- added R27: 62kΩ, ProPrj_Dri-easyedapro:R0402, F.Cu at (-113.0, 43.4)
- added R29: 20kΩ, ProPrj_Dri-easyedapro:R0402, F.Cu at (-113.0, 45.6)
- added R30: 200kΩ, ProPrj_Dri-easyedapro:R0402, F.Cu at (-113.0, 47.7)
- added R31: 10kΩ, ProPrj_Dri-easyedapro:R0402, F.Cu at (-113.0, 49.8)
- added U9: AP64350SP-13, MaslowMerged:AP64350SP_SO-8-EP, F.Cu at (-107.7, 45.6)
- C1: renamed from C7; moved to B.Cu
- C11: renamed from C17; footprint MaslowMerged:C0805 -> ProPrj_Dri-easyedapro:C0402
- C14: renamed from C20; footprint MaslowMerged:C0805 -> ProPrj_Dri-easyedapro:C0603
- C15: renamed from C21; footprint MaslowMerged:C0805 -> ProPrj_Dri-easyedapro:C0603
- C16: renamed from C22; footprint MaslowMerged:C0805 -> ProPrj_Dri-easyedapro:C0603
- C17: renamed from C23; footprint MaslowMerged:C0805 -> ProPrj_Dri-easyedapro:C0603
- C19: renamed from C26; footprint MaslowMerged:C0805 -> ProPrj_Dri-easyedapro:C0402
- C20: renamed from C27; footprint MaslowMerged:C0805 -> ProPrj_Dri-easyedapro:C0402
- C21: renamed from C29; value 470uF -> 22uF; footprint MaslowMerged:CAP-SMD_BD6.3-L6.6-W6.6-LS7.6-RD -> MaslowMerged:C0805
- C22: renamed from C30; footprint MaslowMerged:C0603 -> ProPrj_Dri-easyedapro:C0603
- C26: renamed from C34; footprint MaslowMerged:C0603 -> ProPrj_Dri-easyedapro:C0402
- C3: renamed from C9; footprint MaslowMerged:C0805 -> ProPrj_Dri-easyedapro:C0603
- C34: renamed from C201; footprint ProPrj_Dri-easyedapro:C0402 -> ProPrj_Dri-easyedapro:C0603
- C36: renamed from C203; footprint ProPrj_Dri-easyedapro:C0402 -> ProPrj_Dri-easyedapro:C0603
- C42: renamed from C209; footprint ProPrj_Dri-easyedapro:C0402 -> ProPrj_Dri-easyedapro:C0603
- C45: renamed from C212; footprint ProPrj_Dri-easyedapro:C0402 -> ProPrj_Dri-easyedapro:C0603
- C49: renamed from C216; footprint ProPrj_Dri-easyedapro:C0402 -> ProPrj_Dri-easyedapro:C0603
- C5: renamed from C11; footprint MaslowMerged:C0805 -> ProPrj_Dri-easyedapro:C0603
- C51: renamed from C218; value 100nF/50V -> 100nF
- C54: renamed from C221; footprint ProPrj_Dri-easyedapro:C0402 -> ProPrj_Dri-easyedapro:C0603
- C6: renamed from C12; footprint MaslowMerged:C0805 -> ProPrj_Dri-easyedapro:C0603
- C61: renamed from C230; footprint ProPrj_Dri-easyedapro:C0402 -> ProPrj_Dri-easyedapro:C0603
- C68: renamed from C237; value 100nF/50V -> 100nF
- C8: renamed from C14; footprint MaslowMerged:C0805 -> ProPrj_Dri-easyedapro:C0402
- C9: renamed from C15; footprint MaslowMerged:C0805 -> ProPrj_Dri-easyedapro:C0603
- CN1: value B2B-PH-K-S(LF)(SN) -> B02B-PASK(LF)(SN); footprint MaslowMerged:CONN-TH_B2B-PH-K-S -> MaslowMerged:CONN-TH_B02B-PASK
- CN10: renamed from CN202; moved to B.Cu
- CN11: renamed from CN203; moved to B.Cu
- CN2: renamed from CN3; value B2B-PH-K-S(LF)(SN) -> B02B-PASK(LF)(SN); footprint MaslowMerged:CONN-TH_B2B-PH-K-S -> MaslowMerged:CONN-TH_B02B-PASK
- CN3: renamed from CN4; value B2B-PH-K-S(LF)(SN) -> B02B-PASK(LF)(SN); footprint MaslowMerged:CONN-TH_B2B-PH-K-S -> MaslowMerged:CONN-TH_B02B-PASK
- CN4: renamed from CN5; value B4B-PH-K-S(LF)(SN) -> B04B-PASK(LF)(SN); footprint MaslowMerged:CONN-TH_B4B-PH-K-S -> MaslowMerged:CONN-TH_B04B-PASK
- CN5: renamed from CN9; value B4B-PH-K-S(LF)(SN) -> B04B-PASK(LF)(SN); footprint MaslowMerged:CONN-TH_B4B-PH-K-S -> MaslowMerged:CONN-TH_B04B-PASK
- CN6: renamed from CN10; value B2B-PH-K-S(LF)(SN) -> B02B-PASK(LF)(SN); footprint MaslowMerged:CONN-TH_B2B-PH-K-S -> MaslowMerged:CONN-TH_B02B-PASK
- CN7: renamed from CN11; value B4B-PH-K-S(LF)(SN) -> B04B-PASK(LF)(SN); footprint MaslowMerged:CONN-TH_B4B-PH-K-S -> MaslowMerged:CONN-TH_B04B-PASK
- CN8: renamed from CN12; value B4B-PH-K-S(LF)(SN) -> B04B-PASK(LF)(SN); footprint MaslowMerged:CONN-TH_B4B-PH-K-S -> MaslowMerged:CONN-TH_B04B-PASK
- CN9: renamed from CN201; moved to B.Cu
- L1: renamed from L2; value 33uH -> 4.7uH; footprint MaslowMerged:IND-SMD_L6.0-W6.0 -> Inductor_SMD:L_APV_ANR4030
- R1, R4: footprint MaslowMerged:R0805 -> ProPrj_Dri-easyedapro:R0402
- R10: renamed from R11; footprint MaslowMerged:R0805 -> ProPrj_Dri-easyedapro:R0402
- R11: renamed from R12; footprint MaslowMerged:R0805 -> ProPrj_Dri-easyedapro:R0402
- R12: renamed from R13; footprint MaslowMerged:R0805 -> ProPrj_Dri-easyedapro:R0402
- R13: renamed from R14; footprint MaslowMerged:R0805 -> ProPrj_Dri-easyedapro:R0402
- R19: renamed from R22; footprint MaslowMerged:R0805 -> ProPrj_Dri-easyedapro:R0402
- R20: renamed from R23; footprint MaslowMerged:R0805 -> ProPrj_Dri-easyedapro:R0402
- R21: renamed from R24; footprint MaslowMerged:R0805 -> ProPrj_Dri-easyedapro:R0402
- R25: renamed from R28; value 10K -> 10kΩ; footprint MaslowMerged:R0603 -> ProPrj_Dri-easyedapro:R0402
- R26: renamed from R30; value 10K -> 10kΩ; footprint MaslowMerged:R0603 -> ProPrj_Dri-easyedapro:R0402
- R28: renamed from R32; footprint MaslowMerged:R0805 -> ProPrj_Dri-easyedapro:R0402
- R6: renamed from R7; footprint MaslowMerged:R0805 -> ProPrj_Dri-easyedapro:R0402
- R8: renamed from R9; footprint MaslowMerged:R0805 -> ProPrj_Dri-easyedapro:R0402
- R9: renamed from R10; footprint MaslowMerged:R0805 -> ProPrj_Dri-easyedapro:R0402
- SW1: value DTSL-61N-V-T/R -> TSA002A3512A02; footprint MaslowMerged:SW-SMD_4P-L6.2-W6.4-P4.00-LS7.2 -> ProPrj_Dri-easyedapro:SW-SMD_BZCN_TSA002A35XXX
- U11: renamed from U202; moved to B.Cu
- U12: renamed from U203; moved to B.Cu
- moved SW1 573.6 mm to (-58.8, 73.5), turned to 0 degrees
- moved C10 546.2 mm to (-5.46, -28.2)
- moved C7 540.7 mm to (-8.63, -19.4)
- moved C11 536.3 mm to (-47.4, 1.48)
- moved C17 536.3 mm to (-54.4, -4.49)
- moved C4 536.3 mm to (-59.9, -2.45)
- moved C6 536.3 mm to (-56.7, -2.45)
- moved R10 536.3 mm to (-50.3, 0.47)
- moved R12 536.3 mm to (-50.3, -1.56)
- moved C2 533.0 mm to (-33.0, -45.1)
- moved C3 533.0 mm to (-35.3, -45.1)
- moved C8 533.0 mm to (-36.8, -56.7)
- moved R11 533.0 mm to (-36.7, -54.3)
- moved R9 533.0 mm to (-40.0, -55.5)
- moved U1 526.2 mm to (8.52, -38.3), turned to -12 degrees
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- renumbered C16 to C10, C18 to C12, C19 to C13, C24 to C18, C8 to C2, C31 to C23, C32 to C24, C33 to C25, C40 to C27, C202 to C35, C204 to C37, C205 to C38, C206 to C39, C10 to C4, C207 to C40, C208 to C41, C210 to C43, C211 to C44, C213 to C46, C214 to C47, C215 to C48, C217 to C50, C219 to C52, C220 to C53, C222 to C55, C225 to C56, C226 to C57, C227 to C58, C228 to C59, C229 to C60, C231 to C62, C232 to C63, C233 to C64, C234 to C65, C235 to C66, C236 to C67, C238 to C69, C13 to C7, C239 to C70, C240 to C71, CGQ201 to CGQ1, D2 to D1, D3 to D2, D202 to D3, D204 to D4, IR201 to IR1, LED2 to LED1, LED3 to LED2, LED201 to LED3, R17 to R14, R18 to R15, R19 to R16, R20 to R17, R21 to R18, R25 to R22, R26 to R23, R27 to R24, R201 to R32, R202 to R33, R203 to R34, R204 to R35, R205 to R36, R206 to R37, R207 to R38, R208 to R39, R209 to R40, R210 to R41, R211 to R42, R212 to R43, R213 to R44, R214 to R45, R218 to R46, R219 to R47, R220 to R48, R221 to R49, R6 to R5, R222 to R50, R223 to R51, R224 to R52, R225 to R53, R226 to R54, R227 to R55, R228 to R56, R229 to R57, R230 to R58, R8 to R7, SW201 to SW2, SW202 to SW3, U201 to U10, U5 to U4, U6 to U5, U7 to U6, U9 to U7, U10 to U8, USB2 to USB1, USB201 to USB2
Connections:
- C39 pad 1: VIN -> VCC
- C41 pad 2: VIN -> VCC
- C43 pad 2: VIN -> VCC
- C46 pad 2: VIN -> VCC
- C48 pad 2: VIN -> VCC
- C50 pad 2: VIN -> VCC
- C53 pad 2: VIN -> VCC
- C55 pad 2: VIN -> VCC
- C60 pad 1: VIN -> VCC
- C62 pad 2: VIN -> VCC
- C64 pad 2: VIN -> VCC
- C65 pad 2: VIN -> VCC
- C66 pad 2: VIN -> VCC
- C67 pad 2: VIN -> VCC
- C70 pad 2: VIN -> VCC
- C71 pad 2: VIN -> VCC
- CN10 pad 2: VIN -> VCC
- D1 pad 1: Net-(D2-K) -> VSUP
- D2 pad 1: Net-(D2-K) -> VSUP
- D3 pad 2: VIN -> VCC
- D4 pad 1: VIN_BUCK -> VSUP
- L1 pad 1: Net-(D5-K) -> SW_NODE
- SW1 pad 1: unconnected-(SW1-Pad1) -> Boot
- SW1 pad 2: Boot -> GND
- SW1 pad 4: GND -> unconnected-(SW1-Pad4)
- U10 pad 31: BOARDCOM2 -> BoardCOM1
- U10 pad 32: BOARDCOM1 -> BoardCOM2
- U11 pad 23: VIN -> VCC
- U11 pad 25: VIN -> VCC
- U12 pad 23: VIN -> VCC
- U12 pad 25: VIN -> VCC
- U8 pad 14: BR IN2 -> USBD+
- U8 pad 15: (no net) -> BR IN2
- U8 pad 37: TrinamicRX -> unconnected-(U8-TXD0-Pad37)
- U8 pad 38: (no net) -> TrinamicRX
- U8 pad 39: GND -> TrinamicTX
- U8 pad 40: (no net) -> GND
- U8 pad 41: (no net) -> GND
- USB2 pad 13: unconnected-(USB201-SHELL-Pad13) -> GND
- USB2 pad 14: unconnected-(USB201-SHELL-Pad14) -> GND
Other:
- board size 6.5 x 0.7 mm -> 101.6 x 120.8 mm

Commit message: Main parts placed
Parts:
- C23, C26, C28, C29, C30, C31, C32, C33, D1, D2, D3, L1, R25, R27, R29, R30, R31, SW1, SW2, SW3, U6, U7, U9: moved to B.Cu
- moved C28 159.2 mm to (14.4, 59.1), turned to 90 degrees
- moved C23 129.1 mm to (-5.20, 47.2), turned to 0 degrees
- moved C33 110.5 mm to (-1.90, 91.4), turned to 180 degrees
- moved R30 110.5 mm to (-9.30, 85.9), turned to 180 degrees
- moved L1 110.0 mm to (-4.70, 51.8), turned to 90 degrees
- moved R25 109.5 mm to (6.33, 85.6), turned to 180 degrees
- moved C26 109.5 mm to (6.51, 81.8), turned to 0 degrees
- moved R27 109.1 mm to (-5.17, 60.3), turned to 180 degrees
- moved C31 108.8 mm to (-1.00, 53.3), turned to 180 degrees
- moved C32 107.6 mm to (1.80, 56.8)
- moved R29 106.8 mm to (-7.20, 60.3), turned to 180 degrees
- moved U9 104.7 mm to (-3.60, 56.9), turned to 180 degrees
- moved R31 104.6 mm to (-8.73, 58.7), turned to 180 degrees
- moved SW1 103.2 mm to (35.7, 31.8), turned to 90 degrees
- moved C30 101.1 mm to (-8.85, 57.5), turned to 180 degrees
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Routing:
- net PHC2: track 0.00 -> 53.7 mm
- net PHB2: track 0.00 -> 49.2 mm
- net PHA2: track 0.00 -> 46.1 mm
- net PHC1: track 0.00 -> 37.1 mm
- net PHB1: track 0.00 -> 33.9 mm
- net PHA1: track 0.00 -> 31.1 mm
- net VSUP: track 0.00 -> 25.8 mm, vias 0 -> 1
- net SW_NODE: track 0.00 -> 5.27 mm
- net BoardVersion: track 0.00 -> 4.61 mm
- net COMP: track 0.00 -> 3.42 mm
- net FB: track 0.00 -> 2.70 mm
- net 3V3: track 0.00 -> 2.68 mm, vias 0 -> 2
- net BST: track 0.00 -> 2.03 mm
- net COMP_Z: track 0.00 -> 1.33 mm
- net VCC: vias 0 -> 3
- added copper zone on In2.Cu, net 3V3
- added copper zone on B.Cu, net GND
- added copper zone on F.Cu, net GND
- added copper zone on In1.Cu, net VCC
Other:
- copper layers 2 -> 4

Commit message: Before thermal vias
Parts:
- C12, C14, C4, C6: moved to F.Cu
- C22, C34, C36, C38, C41, C42, C43, C45, C46, C47, C48, C50, C51, C52, C53, C54, C55, C57, C59, C65, C66, C67, C68, C69, D4, R14, R15, R16, R17, R18, R22, R23, R24, R32, R33, R38, R39, R42, R46, R47, R48, R49, R5, R54, R56, R7: moved to B.Cu
- USB2: value TYPE-C 16PIN -> KH-TYPE-C-16P; footprint ProPrj_Dri-easyedapro:USB-C-SMD_TYPE-C-6PIN-2MD-073 -> MaslowMerged:USB-C-SMD_KH-TYPE-C-16P
- moved R9 140.5 mm to (64.9, 37.9), turned to -89.9993 degrees
- moved C8 137.4 mm to (64.9, 35.7), turned to -179.999 degrees
- moved R11 134.9 mm to (62.8, 36.8), turned to -179.999 degrees
- moved C9 126.0 mm to (-5.49, -20.5), turned to 90.0007 degrees
- moved C17 120.5 mm to (58.3, 38.1), turned to -20 degrees
- moved C54 118.4 mm to (36.2, 53.0)
- moved C61 117.6 mm to (-11.3, -15.1), turned to -89.9993 degrees
- moved C42 115.2 mm to (36.2, 55.1)
- moved R12 115.0 mm to (55.4, 43.8), turned to -20 degrees
- moved R10 114.0 mm to (55.8, 42.2), turned to -9.99998 degrees
- moved LED3 113.2 mm to (-6.10, -5.20), turned to -90 degrees
- moved R14 110.1 mm to (8.67, 30.0), turned to 180 degrees
- moved R15 110.1 mm to (8.67, 31.2), turned to 180 degrees
- moved R16 110.1 mm to (8.67, 32.4), turned to 180 degrees
- moved R17 110.1 mm to (8.67, 33.6), turned to 180 degrees
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Connections:
- USB2 pad 2: VBUS -> GND
- USB2 pad 3: unconnected-(USB2-SBU2-Pad3) -> GND
- USB2 pad 4: CC1 -> GND
Routing:
- net 3V3: track 2.68 -> 70.2 mm, vias 2 -> 29
- net GND: track 0.00 -> 51.7 mm, vias 0 -> 7
- net Net-(U2-VCP): track 0.00 -> 17.6 mm, vias 0 -> 1
- net VCC: track 0.00 -> 14.0 mm, vias 3 -> 47
- net Net-(U2-CPH): track 0.00 -> 10.5 mm, vias 0 -> 1
- net PHC2: track 53.7 -> 63.8 mm, vias 0 -> 6
- net PHA1: track 31.1 -> 39.9 mm, vias 0 -> 4
- net PHA2: track 46.1 -> 54.8 mm, vias 0 -> 5
- net FAULT: track 0.00 -> 8.11 mm, vias 0 -> 3
- net Net-(U5-CPH): track 0.00 -> 8.05 mm, vias 0 -> 1
- net Net-(U2-CPL): track 0.00 -> 7.16 mm, vias 0 -> 1
- net PHB1: track 33.9 -> 40.8 mm
- net PHB2: track 49.2 -> 55.9 mm
- net Net-(U3-VCP): track 0.00 -> 6.48 mm
- net NSLEEP: track 0.00 -> 6.32 mm, vias 0 -> 2
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- added copper zone on F.Cu, net BL OUT1
- added copper zone on F.Cu, net BL OUT2
- added copper zone on F.Cu, net BR OUT1
- added copper zone on F.Cu, net BR OUT2
- added copper zone on F.Cu, net TL OUT1
- added copper zone on F.Cu, net TL OUT2
- added copper zone on F.Cu, net TR OUT1
- added copper zone on F.Cu, net TR OUT2
- added copper zone on F.Cu, net VCC

Commit message: Add vias in pins
Routing:
- net VCC: vias 47 -> 55
- net GND: vias 7 -> 67
