File: Unified Control Board/Unified Control Board.kicad_pcb (KiCad board)
At the start: 4 copper layers, 101.6 x 120.8 mm, 167 parts, among them CN1 B02B-PASK(LF)(SN), CN10 B3B-XH-2(LF)(SN), CN11 B3B-XH-2(LF)(SN), CN2 B02B-PASK(LF)(SN), CN3 B02B-PASK(LF)(SN), CN4 B04B-PASK(LF)(SN), CN5 B04B-PASK(LF)(SN), CN6 B02B-PASK(LF)(SN), CN7 B04B-PASK(LF)(SN), CN8 B04B-PASK(LF)(SN), CN9 B3B-XH-2(LF)(SN), SW1 TSA002A3512A02, SW2 TSA002A3512A02, SW3 TSA002A3512A02, U1 XT60PB-M.G.Y, U10 2.4GHz, U11 MP6541A, U12 MP6541A, U2 DRV8876PWPR, U3 DRV8876PWPR, U4 DRV8876PWPR, U5 DRV8876PWPR, U6 TCA9546A, U7 ZDSD01GLGEAG, U8 ESP32-S3-WROOM-1, U9 AP64350SP-13

Commit message: Two wires left to route
Parts:
- removed R6: 1.5kΩ, ProPrj_Dri-easyedapro:R0402
- C62, C64, C70, C71, R43, R57: moved to B.Cu
- moved C39 73.6 mm to (21.5, 8.78), turned to 90 degrees
- moved C17 58.4 mm to (-0.05, 41.1), turned to 90 degrees
- moved R43 37.6 mm to (-30.1, 30.2)
- moved R28 34.0 mm to (26.7, 46.7), turned to 0 degrees
- moved R57 33.8 mm to (-28.9, 30.2)
- moved C8 31.2 mm to (37.4, 50.2), turned to 0.0006614 degrees
- moved R11 29.9 mm to (35.5, 49.0), turned to 0.0006614 degrees
- moved R1 29.6 mm to (35.6, 47.6), turned to 0 degrees
- moved R9 29.5 mm to (37.6, 49.0), turned to -179.999 degrees
- moved C26 28.5 mm to (33.0, 52.5), turned to 90 degrees
- moved R25 27.5 mm to (31.8, 52.2), turned to -90 degrees
- moved R20 26.5 mm to (37.6, 47.6), turned to 180 degrees
- moved C20 24.9 mm to (37.4, 46.5), turned to 0 degrees
- moved C11 21.0 mm to (36.6, 45.3), turned to 0 degrees
- moved R12 20.7 mm to (34.7, 44.1), turned to 0 degrees
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Connections:
- U8 pad 38: TrinamicRX -> unconnected-(U8-IO2-Pad38)
- U8 pad 39: TrinamicTX -> unconnected-(U8-IO1-Pad39)
Routing:
- net FAULT: track 8.11 -> 157.1 mm, vias 3 -> 6
- net Net-(U2-IPROPI): track 2.72 -> 112.6 mm, vias 1 -> 2
- net VAC_CONTROL: track 0.00 -> 105.0 mm, vias 0 -> 2
- net TL IN2: track 3.05 -> 100.9 mm, vias 1 -> 2
- net Net-(U3-IPROPI): track 3.00 -> 100.3 mm, vias 1 -> 2
- net TR IN2: track 3.31 -> 100.2 mm
- net BoardCOM2: track 0.00 -> 95.9 mm, vias 0 -> 5
- net BoardCOM1: track 0.00 -> 95.5 mm, vias 0 -> 5
- net AL2: track 2.59 -> 94.8 mm, vias 1 -> 4
- net TL IN1: track 3.67 -> 95.0 mm, vias 1 -> 2
- net TR IN1: track 3.29 -> 93.5 mm, vias 1 -> 2
- net SDA2: track 2.60 -> 91.9 mm, vias 0 -> 1
- net SCL2: track 2.37 -> 90.3 mm, vias 0 -> 1
- net SCL1: track 2.73 -> 90.2 mm, vias 0 -> 2
- net VBUS: track 0.00 -> 87.0 mm, vias 0 -> 2
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
Commit message: Everything routed?
Routing:
- net DETECTORLED: track 0.00 -> 106.8 mm, vias 0 -> 4
- net BEAMBREAK: track 1.51 -> 92.5 mm, vias 0 -> 4
- net SOC2: track 5.14 -> 36.0 mm
- net Net-(U3-IPROPI): track 100.3 -> 128.7 mm, vias 2 -> 3
- net USB5V: track 58.9 -> 78.0 mm, vias 1 -> 2
- net SOA: track 18.9 -> 28.5 mm, vias 3 -> 2
- net Net-(U2-IPROPI): track 112.6 -> 104.4 mm
- net TR IN1: track 93.5 -> 98.5 mm
- net AH2: track 41.5 -> 46.3 mm, vias 1 -> 2
- net GND: track 65.7 -> 70.1 mm, vias 67 -> 68
- net BH2: track 44.9 -> 49.0 mm
- net SCL0: track 68.8 -> 72.6 mm
- net PHC2: track 63.8 -> 60.4 mm
- net 3V3: track 93.5 -> 96.8 mm, vias 37 -> 38
- net NSLEEP: track 55.0 -> 58.3 mm, vias 4 -> 5
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
Commit message: DRC passing
Routing:
- net 3V3: track 96.8 -> 97.3 mm
Changed lines of the file:
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@@
 	)
 	(via
-		(at -27.3 49.5)
+		(at -27.475 49.2)
 		(size 0.6)
 		(drill 0.3)
@@
 	)
 	(segment
+		(start -42.594685 44.825)
+		(end -42 44.825)
+		(width 0.2)
+		(layer "B.Cu")
+		(net "3V3")
+	)
+	(segment
 		(start -37.2 40.673529)
 		(end -37.598529 40.275)
@@
 	)
 	(segment
+		(start -27.175 49.5)
+		(end -25.767 49.5)
+		(width 0.2)
+		(layer "B.Cu")
+		(net "3V3")
+	)
+	(segment
+		(start -27.475 49.2)
+		(end -27.175 49.5)
+		(width 0.2)
+		(layer "B.Cu")
+		(net "3V3")
+	)
+	(segment
 		(start 27.3 46.7)
 		(end 27.1 46.7)
@@
 	)
 	(segment
+		(start -43.1 45.330315)
+		(end -42.594685 44.825)
+		(width 0.2)
+		(layer "B.Cu")
+		(net "3V3")
+	)
+	(segment
+		(start -27.175 49.5)
+		(end -25.9 49.5)
+		(width 0.2)
+		(layer "B.Cu")
+		(net "3V3")
+	)
+	(segment
+		(start -42 44.825)
+		(end -41.55 44.375)
+		(width 0.2)
+		(layer "B.Cu")
+		(net "3V3")
+	)
+	(segment
 		(start -12.4 54.35)
 		(end -12.4 52.85)
@@
 	)
 	(segment
-		(start -41.581754 43.812069)
-		(end -43.1 45.330315)
+		(start -41.55 44.375)
+		(end -41.55 43.898561)
 		(width 0.2)
 		(layer "B.Cu")
@@
 	)
 	(segment
+		(start -43.1 45.4)
+		(end -43.1 45.330315)
+		(width 0.2)
+		(layer "B.Cu")
+		(net "3V3")
+	)
+	(segment
 		(start 36.9 53.9)
 		(end 36.9 53)
@@
 	)
 	(segment
+		(start -41.55 43.898561)
+		(end -41.463508 43.812069)
+		(width 0.2)
+		(layer "B.Cu")
+		(net "3V3")
+	)
+	(segment
 		(start 8.2344 34.8)
 		(end 8.2344 33.6)
@@
 	)
 	(segment
-		(start -27.3 49.5)
-		(end -25.9 49.5)
-		(width 0.2)
-		(layer "B.Cu")
-		(net "3V3")
-	)
-	(segment
-		(start -27.3 49.5)
-		(end -25.767 49.5)
-		(width 0.2)
-		(layer "B.Cu")
-		(net "3V3")
-	)
-	(segment
 		(start 21.5 34.4)
 		(end 20.2 34.4)
@@
 		(start 17.0001 30.8221)
 		(end 15.2779 30.8221)
-		(width 0.2)
-		(layer "B.Cu")
-		(net "3V3")
-	)
-	(segment
-		(start -43.1 45.330315)
-		(end -43.1 45.4)
 		(width 0.2)
 		(layer "B.Cu")
@@
 	)
 	(segment
+		(start 23.6 -3.8)
+		(end 23.4 -4)
+		(width 0.2)
+		(layer "F.Cu")
+		(net "Net-(U4-CPL)")
+	)
+	(segment
+		(start 23.4 -4)
+		(end 22.150633 -4)
+		(width 0.2)
+		(layer "F.Cu")
+		(net "Net-(U4-CPL)")
+	)
+	(segment
 		(start 23.942896 -2.588037)
 		(end 23.6 -3.8)
@@
 	)
 	(segment
-		(start 23.6 -3.8)
-		(end 21.634171 -4.782388)
-		(width 0.2)
-		(layer "F.Cu")
+		(start 22.150633 -4)
+		(end 21.368245 -4.782388)
+		(width 0.2)
+		(layer "F.Cu")
