File: Unified Control Board/Unified Control Board.kicad_pcb (KiCad board)
At the start: 4 copper layers, 101.6 x 120.8 mm, 166 parts, among them CN1 B02B-PASK(LF)(SN), CN10 B3B-XH-2(LF)(SN), CN11 B3B-XH-2(LF)(SN), CN2 B02B-PASK(LF)(SN), CN3 B02B-PASK(LF)(SN), CN4 B04B-PASK(LF)(SN), CN5 B04B-PASK(LF)(SN), CN6 B02B-PASK(LF)(SN), CN7 B04B-PASK(LF)(SN), CN8 B04B-PASK(LF)(SN), CN9 B3B-XH-2(LF)(SN), SW1 TSA002A3512A02, SW2 TSA002A3512A02, SW3 TSA002A3512A02, U1 XT60PB-M.G.Y, U10 2.4GHz, U11 MP6541A, U12 MP6541A, U2 DRV8876PWPR, U3 DRV8876PWPR, U4 DRV8876PWPR, U5 DRV8876PWPR, U6 TCA9546A, U7 ZDSD01GLGEAG, U8 ESP32-S3-WROOM-1, U9 AP64350SP-13

Commit message: Seems good to order
Parts:
- added FID1: Fiducial, Fiducial:Fiducial_1mm_Mask2mm, F.Cu at (-28.0, -9.00)
- added FID2: Fiducial, Fiducial:Fiducial_1mm_Mask2mm, F.Cu at (31.0, 11.0)
- added FID3: Fiducial, Fiducial:Fiducial_1mm_Mask2mm, F.Cu at (20.0, 69.0)
- added FID4: Fiducial, Fiducial:Fiducial_1mm_Mask2mm, B.Cu at (-43.0, 48.0)
- added FID5: Fiducial, Fiducial:Fiducial_1mm_Mask2mm, B.Cu at (7.00, -33.0)
- added FID6: Fiducial, Fiducial:Fiducial_1mm_Mask2mm, B.Cu at (43.0, 46.0)
Routing:
- net AL2: track 94.8 -> 70.4 mm, vias 4 -> 3
- net FAULT: track 157.5 -> 149.2 mm
- net USB5V: track 78.0 -> 74.1 mm
- net GND: track 70.1 -> 72.4 mm, vias 68 -> 82
- net BoardCOM2: track 95.9 -> 94.1 mm
- net Net-(CGQ1-A): track 0.00 -> 1.40 mm
- net TL IN1: track 97.9 -> 96.8 mm
- net SCL0: track 72.6 -> 73.7 mm
- net SDA0: track 64.8 -> 65.6 mm
- net PHC1: track 41.9 -> 41.3 mm
- net NFAULT: track 33.5 -> 32.9 mm
- net BR IN1: track 63.0 -> 62.9 mm, vias 1 -> 0
- net VSUP: vias 1 -> 0
- net TR IN2: vias 1 -> 0
- net PHA2: vias 3 -> 2
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