File: Unified Control Board/Unified Control Board.kicad_sch (KiCad schematic)
At the start: 171 parts, among them CN1 B2B-PH-K-S(LF)(SN), CN10 B2B-PH-K-S(LF)(SN), CN11 B4B-PH-K-S(LF)(SN), CN12 B4B-PH-K-S(LF)(SN), CN201 B3B-XH-2(LF)(SN), CN202 B3B-XH-2(LF)(SN), CN203 B3B-XH-2(LF)(SN), CN3 B2B-PH-K-S(LF)(SN), CN4 B2B-PH-K-S(LF)(SN), CN5 B4B-PH-K-S(LF)(SN), CN9 B4B-PH-K-S(LF)(SN), SW1 DTSL-61N-V-T/R, SW201 TSA002A3512A02, SW202 TSA002A3512A02, U1 XT60PB-M.G.Y, U10 ESP32-S3-WROOM-1, U16 LM2596R-3.3, U2 DRV8876PWPR, U201 2.4GHz, U202 MP6541A, U203 MP6541A, U204 MP2459GJ-Z, U3 DRV8876PWPR, U5 DRV8876PWPR, U6 DRV8876PWPR, U7 TCA9546A, U9 ZDSD01GLGEAG

Commit message: Merging nets and voltage regulators
Parts:
- removed C223: 10uF/50V, ProPrj_Dri-easyedapro:C0805, symbol ProPrj_Dri-easyedapro:GRM21BR61H106KE43L
- removed C224: 100nF/50V, ProPrj_Dri-easyedapro:C0603, symbol ProPrj_Dri-easyedapro:CL05B104KB54PNC
- removed D1: verde, MaslowMerged:LED0603-R-RD, symbol 19-217/GHC-YR1S2/3T
- removed D201, D203: SS36, Diode_SMD:D_SMA, symbol ProPrj_Dri-easyedapro:SS36
- removed D5: RB050L-60TE25, MaslowMerged:SMA_L4.3-W2.7-LS5.1-RD, symbol RB050L-60TE25
- removed H1: 210S-2*5P L=11.6MMGold-plated black, MaslowMerged:HDR-TH_10P-P2.54-V-M-R2-C5-S2.54, symbol 210S-2*5P L=11.6MMGold-plated black
- removed H201: B-2100N10P-B110, ProPrj_Dri-easyedapro:HDR-SMD_10P-P2.54-V-M-R2-C5-S2.54-LS7.3, symbol ProPrj_Dri-easyedapro:210SMT-2*5P Gold-plated black
- removed L201: 47uH, Inductor_SMD:L_Bourns_SRN6045TA, symbol ProPrj_Dri-easyedapro:PRS3015-470MT
- removed R15: 120Ω, MaslowMerged:R0603, symbol 0603WAF1200T5E_2
- removed R215: 124kΩ, ProPrj_Dri-easyedapro:R0402, symbol ProPrj_Dri-easyedapro:0402WGF1003TCE
- removed R216: 40.2kΩ, ProPrj_Dri-easyedapro:R0402, symbol ProPrj_Dri-easyedapro:0402WGF1002TCE
- removed R217: 100kΩ, ProPrj_Dri-easyedapro:R0402, symbol ProPrj_Dri-easyedapro:0402WGF1003TCE
- removed SW1: DTSL-61N-V-T/R, MaslowMerged:SW-SMD_4P-L6.2-W6.4-P4.00-LS7.2, symbol DTSL-61N-V-T/R
- removed U16: LM2596R-3.3, MaslowMerged:TO-263-5_L10.2-W8.6-P1.70-LS14.4-TL, symbol LM2596R-3.3
- removed U204: MP2459GJ-Z, Package_TO_SOT_SMD:SOT-23-6, symbol ProPrj_Dri-easyedapro:MP2459
- added C28: 680uF, MaslowMerged:CAP-SMD_BD10.0-L10.3-W10.3-LS10.9-FD, symbol GVM1V681M1010
- added C29: 3.3nF, ProPrj_Dri-easyedapro:C0402, symbol ProPrj_Dri-easyedapro:0402CG220J500NT
- added C30: 68pF, ProPrj_Dri-easyedapro:C0402, symbol ProPrj_Dri-easyedapro:0402CG220J500NT
- added C31: 100nF, ProPrj_Dri-easyedapro:C0603, symbol ProPrj_Dri-easyedapro:0402CG220J500NT
- added C32: 10uF, ProPrj_Dri-easyedapro:C0805, symbol ProPrj_Dri-easyedapro:GRM21BR61H106KE43L
- added C33: 22uF, ProPrj_Dri-easyedapro:C0805, symbol ProPrj_Dri-easyedapro:GRM21BR61H106KE43L
- added R27: 62kΩ, ProPrj_Dri-easyedapro:R0402, symbol ProPrj_Dri-easyedapro:0402WGF1002TCE
- added R29: 20kΩ, ProPrj_Dri-easyedapro:R0402, symbol ProPrj_Dri-easyedapro:0402WGF1002TCE
- added R30: 200kΩ, ProPrj_Dri-easyedapro:R0402, symbol ProPrj_Dri-easyedapro:0402WGF1002TCE
- added R31: 10kΩ, ProPrj_Dri-easyedapro:R0402, symbol ProPrj_Dri-easyedapro:0402WGF1002TCE
- added SW1: TSA002A3512A02, ProPrj_Dri-easyedapro:SW-SMD_BZCN_TSA002A35XXX, symbol ProPrj_Dri-easyedapro:TSA002A3512A02
- added U9: AP64350SP-13, MaslowMerged:AP64350SP_SO-8-EP, symbol MaslowMerged:AP64350
- C1: renamed from C7; MPN (none) -> RT1J220M0607; Manufacturer Part RVT1J220M0607 -> (none); Supplier Part C72501 -> C267472
- C10: renamed from C16; MPN (none) -> RT1J220M0607; Manufacturer Part RVT1J220M0607 -> (none); Supplier Part C72501 -> C267472
- C11: renamed from C17; footprint MaslowMerged:C0805 -> ProPrj_Dri-easyedapro:C0402; MPN (none) -> CL05A105KA5NQNC; Manufacturer Part CL21B105KBFNNNE -> (none); Supplier Part C28323 -> C52923
- C12: renamed from C18; MPN (none) -> CL21B223KBANNNC; Manufacturer Part CL21B223KBANNNC -> (none)
- C13: renamed from C19; MPN (none) -> CL21B223KBANNNC; Manufacturer Part CL21B223KBANNNC -> (none)
- C14: renamed from C20; footprint MaslowMerged:C0805 -> ProPrj_Dri-easyedapro:C0603; MPN (none) -> CC0603KRX7R9BB104; Manufacturer Part CC0805KRX7R9BB104 -> (none); Supplier Part C49678 -> C14663
- C15: renamed from C21; footprint MaslowMerged:C0805 -> ProPrj_Dri-easyedapro:C0603; MPN (none) -> CC0603KRX7R9BB104; Manufacturer Part CC0805KRX7R9BB104 -> (none); Supplier Part C49678 -> C14663
- C16: renamed from C22; footprint MaslowMerged:C0805 -> ProPrj_Dri-easyedapro:C0603; MPN (none) -> CC0603KRX7R9BB104; Manufacturer Part CC0805KRX7R9BB104 -> (none); Supplier Part C49678 -> C14663
- C17: renamed from C23; footprint MaslowMerged:C0805 -> ProPrj_Dri-easyedapro:C0603; MPN (none) -> CC0603KRX7R9BB104; Manufacturer Part CC0805KRX7R9BB104 -> (none); Supplier Part C49678 -> C14663
- C18: renamed from C24; MPN (none) -> RT1J220M0607; Manufacturer Part RVT1J220M0607 -> (none); Supplier Part C72501 -> C267472
- C19: renamed from C26; footprint MaslowMerged:C0805 -> ProPrj_Dri-easyedapro:C0402; MPN (none) -> CL05A105KA5NQNC; Manufacturer Part CL21B105KBFNNNE -> (none); Supplier Part C28323 -> C52923
- C2: renamed from C8; MPN (none) -> CL21B223KBANNNC; Manufacturer Part CL21B223KBANNNC -> (none)
- C20: renamed from C27; footprint MaslowMerged:C0805 -> ProPrj_Dri-easyedapro:C0402; MPN (none) -> CL05A105KA5NQNC; Manufacturer Part CL21B105KBFNNNE -> (none); Supplier Part C28323 -> C52923
- C21: renamed from C29; value 470uF -> 22uF; footprint MaslowMerged:CAP-SMD_BD6.3-L6.6-W6.6-LS7.6-RD -> MaslowMerged:C0805; MPN (none) -> CL21A226MAQNNNE; Manufacturer ROQANG(容强) -> Samsung Electro-Mechanics; Manufacturer Part RVT1C471M0607 -> (none); Supplier Part C2977552 -> C45783
- C22: renamed from C30; footprint MaslowMerged:C0603 -> ProPrj_Dri-easyedapro:C0603; MPN (none) -> CC0603KRX7R9BB104; Manufacturer Part CC0603KRX7R9BB104 -> (none)
- C23: renamed from C31; MPN (none) -> CL21A106KAYNNNE; Manufacturer Part CL21A106KAYNNNE -> (none)
- C24: renamed from C32; MPN (none) -> CC0603JRNPO9BN220; Manufacturer Part CC0603JRNPO9BN220 -> (none)
- C25: renamed from C33; MPN (none) -> CC0603JRNPO9BN220; Manufacturer Part CC0603JRNPO9BN220 -> (none)
- C26: renamed from C34; footprint MaslowMerged:C0603 -> ProPrj_Dri-easyedapro:C0402; MPN (none) -> CL05A105KA5NQNC; Manufacturer SAMSUNG -> SAMSUNG(三星); Manufacturer Part CL10A105KA8NNNC -> (none); Supplier Part C5673 -> C52923
- C27: renamed from C40; MPN (none) -> GVM1V681M1010; Manufacturer Part GVM1V681M1010 -> (none)
- C3: renamed from C9; footprint MaslowMerged:C0805 -> ProPrj_Dri-easyedapro:C0603; MPN (none) -> CC0603KRX7R9BB104; Manufacturer Part CC0805KRX7R9BB104 -> (none); Supplier Part C49678 -> C14663
- C34: renamed from C201; footprint ProPrj_Dri-easyedapro:C0402 -> ProPrj_Dri-easyedapro:C0603; MPN (none) -> CC0603KRX7R9BB104; Manufacturer SAMSUNG(三星) -> YAGEO(国巨); Manufacturer Part CL05B104KB54PNC -> (none); Supplier Part C307331 -> C14663
- C35: renamed from C202; MPN (none) -> 0402B102K500NT; Manufacturer Samsung Electro-Mechanics -> FH(Guangdong Fenghua); Manufacturer Part CL05B102KB5NNNC -> (none); Supplier Part C14442 -> C1523
- C36: renamed from C203; footprint ProPrj_Dri-easyedapro:C0402 -> ProPrj_Dri-easyedapro:C0603; MPN (none) -> CC0603KRX7R9BB104; Manufacturer SAMSUNG(三星) -> YAGEO(国巨); Manufacturer Part CL05B104KB54PNC -> (none); Supplier Part C307331 -> C14663
- C37: renamed from C204; MPN (none) -> 0402B102K500NT; Manufacturer Samsung Electro-Mechanics -> FH(Guangdong Fenghua); Manufacturer Part CL05B102KB5NNNC -> (none); Supplier Part C14442 -> C1523
- C38: renamed from C205; MPN (none) -> 0402B102K500NT; Manufacturer Samsung Electro-Mechanics -> FH(Guangdong Fenghua); Manufacturer Part CL05B102KB5NNNC -> (none); Supplier Part C14442 -> C1523
- C39: renamed from C206; MPN (none) -> ERS1VM221F12OT; Manufacturer Part ERS1VM221F12OT -> (none)
- C4: renamed from C10; MPN (none) -> CL21B223KBANNNC; Manufacturer Part CL21B223KBANNNC -> (none)
- C40: renamed from C207; MPN (none) -> CL05A105KA5NQNC; Manufacturer Part CL05A105KA5NQNC -> (none)
- C41: renamed from C208; MPN (none) -> GRM21BR61H106KE43L; Manufacturer Part GRM21BR61H106KE43L -> (none)
- C42: renamed from C209; footprint ProPrj_Dri-easyedapro:C0402 -> ProPrj_Dri-easyedapro:C0603; MPN (none) -> CC0603KRX7R9BB104; Manufacturer SAMSUNG(三星) -> YAGEO(国巨); Manufacturer Part CL05B104KB54PNC -> (none); Supplier Part C307331 -> C14663
- C43: renamed from C210; MPN (none) -> GRM21BR61H106KE43L; Manufacturer Part GRM21BR61H106KE43L -> (none)
- C44: renamed from C211; MPN (none) -> CL05A105KA5NQNC; Manufacturer Part CL05A105KA5NQNC -> (none)
- C45: renamed from C212; footprint ProPrj_Dri-easyedapro:C0402 -> ProPrj_Dri-easyedapro:C0603; MPN (none) -> CC0603KRX7R9BB104; Manufacturer SAMSUNG(三星) -> YAGEO(国巨); Manufacturer Part CL05B104KB54PNC -> (none); Supplier Part C307331 -> C14663
- C46: renamed from C213; MPN (none) -> GRM21BR61H106KE43L; Manufacturer Part GRM21BR61H106KE43L -> (none)
- C47: renamed from C214; MPN (none) -> CL05A105KA5NQNC; Manufacturer Part CL05A105KA5NQNC -> (none)
- C48: renamed from C215; MPN (none) -> GRM21BR61H106KE43L; Manufacturer Part GRM21BR61H106KE43L -> (none)
- C49: renamed from C216; footprint ProPrj_Dri-easyedapro:C0402 -> ProPrj_Dri-easyedapro:C0603; MPN (none) -> CC0603KRX7R9BB104; Manufacturer SAMSUNG(三星) -> YAGEO(国巨); Manufacturer Part CL05B104KB54PNC -> (none); Supplier Part C307331 -> C14663
- C5: renamed from C11; footprint MaslowMerged:C0805 -> ProPrj_Dri-easyedapro:C0603; MPN (none) -> CC0603KRX7R9BB104; Manufacturer Part CC0805KRX7R9BB104 -> (none); Supplier Part C49678 -> C14663
- C50: renamed from C217; MPN (none) -> CL10B105KB8NQNC; Manufacturer Part CL10B105KO8NNNC -> (none); Supplier Part C59782 -> C5199872
- C51: renamed from C218; value 100nF/50V -> 100nF; MPN (none) -> CC0603KRX7R9BB104; Manufacturer Samsung Electro-Mechanics -> YAGEO(国巨); Manufacturer Part CL10B104KB8NNNC -> (none); Supplier Part C1591 -> C14663
- C52: renamed from C219; MPN (none) -> CL21A475KAQNNNE; Manufacturer Taiyo Yuden -> Samsung Electro-Mechanics; Manufacturer Part EMK212B7475KG-T -> (none); Supplier Part C92762 -> C1779
- C53: renamed from C220; MPN (none) -> GRM21BR61H106KE43L; Manufacturer Part GRM21BR61H106KE43L -> (none)
- C54: renamed from C221; footprint ProPrj_Dri-easyedapro:C0402 -> ProPrj_Dri-easyedapro:C0603; MPN (none) -> CC0603KRX7R9BB104; Manufacturer SAMSUNG(三星) -> YAGEO(国巨); Manufacturer Part CL05B104KB54PNC -> (none); Supplier Part C307331 -> C14663
- C55: renamed from C222; MPN (none) -> GRM21BR61H106KE43L; Manufacturer Part GRM21BR61H106KE43L -> (none)
- C56: renamed from C225; MPN (none) -> CL21A226MAQNNNE; Manufacturer Murata -> Samsung Electro-Mechanics; Manufacturer Part GRM219R61C226ME15L -> (none); Supplier Part C162295 -> C45783
- C57: renamed from C226; MPN (none) -> 0402B102K500NT; Manufacturer Samsung Electro-Mechanics -> FH(Guangdong Fenghua); Manufacturer Part CL05B102KB5NNNC -> (none); Supplier Part C14442 -> C1523
- C58: renamed from C227; MPN (none) -> 0402B102K500NT; Manufacturer Samsung Electro-Mechanics -> FH(Guangdong Fenghua); Manufacturer Part CL05B102KB5NNNC -> (none); Supplier Part C14442 -> C1523
- C59: renamed from C228; MPN (none) -> 0402B102K500NT; Manufacturer Samsung Electro-Mechanics -> FH(Guangdong Fenghua); Manufacturer Part CL05B102KB5NNNC -> (none); Supplier Part C14442 -> C1523
- C6: renamed from C12; footprint MaslowMerged:C0805 -> ProPrj_Dri-easyedapro:C0603; MPN (none) -> CC0603KRX7R9BB104; Manufacturer Part CC0805KRX7R9BB104 -> (none); Supplier Part C49678 -> C14663
- C60: renamed from C229; MPN (none) -> ERS1VM221F12OT; Manufacturer Part ERS1VM221F12OT -> (none)
- C61: renamed from C230; footprint ProPrj_Dri-easyedapro:C0402 -> ProPrj_Dri-easyedapro:C0603; MPN (none) -> CC0603KRX7R9BB104; Manufacturer SAMSUNG(三星) -> YAGEO(国巨); Manufacturer Part CL05B104KB54PNC -> (none); Supplier Part C307331 -> C14663
- C62: renamed from C231; MPN (none) -> GRM21BR61H106KE43L; Manufacturer Part GRM21BR61H106KE43L -> (none)
- C63: renamed from C232; MPN (none) -> CL21A226MAQNNNE; Manufacturer Murata Electronics -> Samsung Electro-Mechanics; Manufacturer Part GRM219R61C226ME15L -> (none); Supplier Part C162295 -> C45783
- C64: renamed from C233; MPN (none) -> GRM21BR61H106KE43L; Manufacturer Part GRM21BR61H106KE43L -> (none)
- C65: renamed from C234; MPN (none) -> GRM21BR61H106KE43L; Manufacturer Part GRM21BR61H106KE43L -> (none)
- C66: renamed from C235; MPN (none) -> GRM21BR61H106KE43L; Manufacturer Part GRM21BR61H106KE43L -> (none)
- C67: renamed from C236; MPN (none) -> CL10B105KB8NQNC; Manufacturer Part CL10B105KO8NNNC -> (none); Supplier Part C59782 -> C5199872
- C68: renamed from C237; value 100nF/50V -> 100nF; MPN (none) -> CC0603KRX7R9BB104; Manufacturer Samsung Electro-Mechanics -> YAGEO(国巨); Manufacturer Part CL10B104KB8NNNC -> (none); Supplier Part C1591 -> C14663
- C69: renamed from C238; MPN (none) -> CL21A475KAQNNNE; Manufacturer Taiyo Yuden -> Samsung Electro-Mechanics; Manufacturer Part EMK212B7475KG-T -> (none); Supplier Part C92762 -> C1779
- C7: renamed from C13; MPN (none) -> RT1J220M0607; Manufacturer Part RVT1J220M0607 -> (none); Supplier Part C72501 -> C267472
- C70: renamed from C239; MPN (none) -> GRM21BR61H106KE43L; Manufacturer Part GRM21BR61H106KE43L -> (none)
- C71: renamed from C240; MPN (none) -> GRM21BR61H106KE43L; Manufacturer Part GRM21BR61H106KE43L -> (none)
- C8: renamed from C14; footprint MaslowMerged:C0805 -> ProPrj_Dri-easyedapro:C0402; MPN (none) -> CL05A105KA5NQNC; Manufacturer Part CL21B105KBFNNNE -> (none); Supplier Part C28323 -> C52923
- C9: renamed from C15; footprint MaslowMerged:C0805 -> ProPrj_Dri-easyedapro:C0603; MPN (none) -> CC0603KRX7R9BB104; Manufacturer Part CC0805KRX7R9BB104 -> (none); Supplier Part C49678 -> C14663
- CGQ1: renamed from CGQ201; MPN (none) -> IR12-21C/TR8; Manufacturer Part IR12-21C/TR8 -> (none)
- CN1: value B2B-PH-K-S(LF)(SN) -> B02B-PASK(LF)(SN); footprint MaslowMerged:CONN-TH_B2B-PH-K-S -> MaslowMerged:CONN-TH_B02B-PASK; MPN (none) -> B02B-PASK(LF)(SN); Manufacturer Part B2B-PH-K-S(LF)(SN) -> (none); Supplier Part C131337 -> C158050
- CN10: renamed from CN202; MPN (none) -> B3B-XH-2(LF)(SN); Manufacturer Part B3B-XH-2(LF)(SN) -> (none)
- CN11: renamed from CN203; MPN (none) -> B3B-XH-2(LF)(SN); Manufacturer Part B3B-XH-2(LF)(SN) -> (none)
- CN2: renamed from CN3; value B2B-PH-K-S(LF)(SN) -> B02B-PASK(LF)(SN); footprint MaslowMerged:CONN-TH_B2B-PH-K-S -> MaslowMerged:CONN-TH_B02B-PASK; MPN (none) -> B02B-PASK(LF)(SN); Manufacturer Part B2B-PH-K-S(LF)(SN) -> (none); Supplier Part C131337 -> C158050
- CN3: renamed from CN4; value B2B-PH-K-S(LF)(SN) -> B02B-PASK(LF)(SN); footprint MaslowMerged:CONN-TH_B2B-PH-K-S -> MaslowMerged:CONN-TH_B02B-PASK; MPN (none) -> B02B-PASK(LF)(SN); Manufacturer Part B2B-PH-K-S(LF)(SN) -> (none); Supplier Part C131337 -> C158050
- CN4: renamed from CN5; value B4B-PH-K-S(LF)(SN) -> B04B-PASK(LF)(SN); footprint MaslowMerged:CONN-TH_B4B-PH-K-S -> MaslowMerged:CONN-TH_B04B-PASK; MPN (none) -> B04B-PASK(LF)(SN); Manufacturer Part B4B-PH-K-S(LF)(SN) -> (none); Supplier Part C131334 -> C265078
- CN5: renamed from CN9; value B4B-PH-K-S(LF)(SN) -> B04B-PASK(LF)(SN); footprint MaslowMerged:CONN-TH_B4B-PH-K-S -> MaslowMerged:CONN-TH_B04B-PASK; MPN (none) -> B04B-PASK(LF)(SN); Manufacturer Part B4B-PH-K-S(LF)(SN) -> (none); Supplier Part C131334 -> C265078
- CN6: renamed from CN10; value B2B-PH-K-S(LF)(SN) -> B02B-PASK(LF)(SN); footprint MaslowMerged:CONN-TH_B2B-PH-K-S -> MaslowMerged:CONN-TH_B02B-PASK; MPN (none) -> B02B-PASK(LF)(SN); Manufacturer Part B2B-PH-K-S(LF)(SN) -> (none); Supplier Part C131337 -> C158050
- CN7: renamed from CN11; value B4B-PH-K-S(LF)(SN) -> B04B-PASK(LF)(SN); footprint MaslowMerged:CONN-TH_B4B-PH-K-S -> MaslowMerged:CONN-TH_B04B-PASK; MPN (none) -> B04B-PASK(LF)(SN); Manufacturer Part B4B-PH-K-S(LF)(SN) -> (none); Supplier Part C131334 -> C265078
- CN8: renamed from CN12; value B4B-PH-K-S(LF)(SN) -> B04B-PASK(LF)(SN); footprint MaslowMerged:CONN-TH_B4B-PH-K-S -> MaslowMerged:CONN-TH_B04B-PASK; MPN (none) -> B04B-PASK(LF)(SN); Manufacturer Part B4B-PH-K-S(LF)(SN) -> (none); Supplier Part C131334 -> C265078
- CN9: renamed from CN201; MPN (none) -> B3B-XH-2(LF)(SN); Manufacturer Part B3B-XH-2(LF)(SN) -> (none)
- D1: renamed from D2; MPN (none) -> SS14; Manufacturer Part SS14 -> (none)
- D2: renamed from D3; MPN (none) -> SS14; Manufacturer Part SS14 -> (none)
- D3: renamed from D202; MPN (none) -> SMCJ24A; Manufacturer Part SMCJ24A -> (none)
- D4: renamed from D204; MPN (none) -> SS36; Manufacturer Part SS36 -> (none)
- IR1: renamed from IR201; MPN (none) -> PT12-21C/TR8; Manufacturer Part PT12-21C/TR8 -> (none)
- L1: renamed from L2; value 33uH -> 4.7uH; footprint MaslowMerged:IND-SMD_L6.0-W6.0 -> Inductor_SMD:L_APV_ANR4030; MPN (none) -> FNR4030S4R7MT; Manufacturer CENKER -> CODACA; Manufacturer Part CKCS6045-33uH/M -> (none); Supplier Part C354635 -> C167874
- LED1: renamed from LED2; MPN (none) -> KT-0603R; Manufacturer EVERLIGHT(台湾亿光) -> Hubei KENTO Elec; Manufacturer Part 19-217/R6C-AL1M2VY/3T -> (none); Supplier Part C72044 -> C2286
- LED2: renamed from LED3; MPN (none) -> NCD0603B1; Manufacturer Part NCD0603B1 -> (none)
- LED3: renamed from LED201; MPN (none) -> KT-0603YG; Manufacturer Part KT-0603YG -> (none)
- R1: footprint MaslowMerged:R0805 -> ProPrj_Dri-easyedapro:R0402; MPN (none) -> 0402WGF1501TCE; Manufacturer Part 0805W8F1501T5E -> (none); Supplier Part C4310 -> C25867
- R10: renamed from R11; footprint MaslowMerged:R0805 -> ProPrj_Dri-easyedapro:R0402; MPN (none) -> 0402WGF1002TCE; Manufacturer Part 0805W8F1002T5E -> (none); Supplier Part C17414 -> C25744
- R11: renamed from R12; footprint MaslowMerged:R0805 -> ProPrj_Dri-easyedapro:R0402; MPN (none) -> 0402WGF1501TCE; Manufacturer Part 0805W8F1501T5E -> (none); Supplier Part C4310 -> C25867
- R12: renamed from R13; footprint MaslowMerged:R0805 -> ProPrj_Dri-easyedapro:R0402; MPN (none) -> 0402WGF1501TCE; Manufacturer Part 0805W8F1501T5E -> (none); Supplier Part C4310 -> C25867
- R13: renamed from R14; footprint MaslowMerged:R0805 -> ProPrj_Dri-easyedapro:R0402; MPN (none) -> 0402WGF5101TCE; Manufacturer Part 0805W8F5101T5E -> (none); Supplier Part C27834 -> C25905
- R14: renamed from R17; MPN (none) -> 0402WGF1001TCE; Manufacturer Part 0402WGF1001TCE -> (none)
- R15: renamed from R18; MPN (none) -> 0402WGF1001TCE; Manufacturer Part 0402WGF1001TCE -> (none)
- R16: renamed from R19; MPN (none) -> 0402WGF1001TCE; Manufacturer Part 0402WGF1001TCE -> (none)
- R17: renamed from R20; MPN (none) -> 0402WGF1001TCE; Manufacturer Part 0402WGF1001TCE -> (none)
- R18: renamed from R21; MPN (none) -> 0402WGF1001TCE; Manufacturer Part 0402WGF1001TCE -> (none)
- R19: renamed from R22; footprint MaslowMerged:R0805 -> ProPrj_Dri-easyedapro:R0402; MPN (none) -> 0402WGF1002TCE; Manufacturer Part 0805W8F1002T5E -> (none); Supplier Part C17414 -> C25744
- R2, R3: MPN (none) -> 0603WAF1200T5E; Manufacturer Part 0603WAF1200T5E -> (none)
- R20: renamed from R23; footprint MaslowMerged:R0805 -> ProPrj_Dri-easyedapro:R0402; MPN (none) -> 0402WGF1002TCE; Manufacturer Part 0805W8F1002T5E -> (none); Supplier Part C17414 -> C25744
- R21: renamed from R24; footprint MaslowMerged:R0805 -> ProPrj_Dri-easyedapro:R0402; MPN (none) -> 0402WGF1501TCE; Manufacturer Part 0805W8F1501T5E -> (none); Supplier Part C4310 -> C25867
- R22: renamed from R25; MPN (none) -> 0402WGF1001TCE; Manufacturer Part 0402WGF1001TCE -> (none)
- R23: renamed from R26; MPN (none) -> 0402WGF1001TCE; Manufacturer Part 0402WGF1001TCE -> (none)
- R24: renamed from R27; MPN (none) -> 0402WGF1001TCE; Manufacturer Part 0402WGF1001TCE -> (none)
- R25: renamed from R28; value 10K -> 10kΩ; footprint MaslowMerged:R0603 -> ProPrj_Dri-easyedapro:R0402; MPN (none) -> 0402WGF1002TCE; Manufacturer YAGEO -> UNI-ROYAL(厚声); Manufacturer Part RC0603JR-0710KL -> (none); Supplier Part C99198 -> C25744
- R26: renamed from R30; value 10K -> 10kΩ; footprint MaslowMerged:R0603 -> ProPrj_Dri-easyedapro:R0402; MPN (none) -> 0402WGF1002TCE; Manufacturer YAGEO -> UNI-ROYAL(厚声); Manufacturer Part RC0603JR-0710KL -> (none); Supplier Part C99198 -> C25744
- R28: renamed from R32; footprint MaslowMerged:R0805 -> ProPrj_Dri-easyedapro:R0402; MPN (none) -> 0402WGF1002TCE; Manufacturer Part 0805W8F1002T5E -> (none); Supplier Part C17414 -> C25744
- R32: renamed from R201; MPN (none) -> 0402WGF3301TCE; Manufacturer Yageo -> UNI-ROYAL(厚声); Manufacturer Part RC0402FR-073K3L -> (none); Supplier Part C137992 -> C25890
- R33: renamed from R202; MPN (none) -> 0402WGF3301TCE; Manufacturer Yageo -> UNI-ROYAL(厚声); Manufacturer Part RC0402FR-073K3L -> (none); Supplier Part C137992 -> C25890
- R34: renamed from R203; MPN (none) -> 0402WGF3301TCE; Manufacturer Yageo -> UNI-ROYAL(厚声); Manufacturer Part RC0402FR-073K3L -> (none); Supplier Part C137992 -> C25890
- R35: renamed from R204; MPN (none) -> 0402WGF3301TCE; Manufacturer Yageo -> UNI-ROYAL(厚声); Manufacturer Part RC0402FR-073K3L -> (none); Supplier Part C137992 -> C25890
- R36: renamed from R205; MPN (none) -> 0402WGF3301TCE; Manufacturer Yageo -> UNI-ROYAL(厚声); Manufacturer Part RC0402FR-073K3L -> (none); Supplier Part C137992 -> C25890
- R37: renamed from R206; MPN (none) -> 0402WGF3301TCE; Manufacturer Yageo -> UNI-ROYAL(厚声); Manufacturer Part RC0402FR-073K3L -> (none); Supplier Part C137992 -> C25890
- R38: renamed from R207; MPN (none) -> 0402WGF1002TCE; Manufacturer Part 0402WGF1002TCE -> (none)
- R39: renamed from R208; MPN (none) -> 0402WGF1002TCE; Manufacturer Part 0402WGF1002TCE -> (none)
- R4: footprint MaslowMerged:R0805 -> ProPrj_Dri-easyedapro:R0402; MPN (none) -> 0402WGF5101TCE; Manufacturer Part 0805W8F5101T5E -> (none); Supplier Part C27834 -> C25905
- R40: renamed from R209; MPN (none) -> 0402WGF3300TCE; Manufacturer Part 0402WGF3300TCE -> (none)
- R41: renamed from R210; MPN (none) -> 0402WGF3300TCE; Manufacturer Part 0402WGF3300TCE -> (none)
- R42: renamed from R211; MPN (none) -> 0402WGF3300TCE; Manufacturer Part 0402WGF3300TCE -> (none)
- R43: renamed from R212; MPN (none) -> 0402WGF5101TCE; Manufacturer Part 0402WGF5101TCE -> (none)
- R44: renamed from R213; MPN (none) -> 0402WGF1000TCE; Manufacturer Part 0402WGF1000TCE -> (none)
- R45: renamed from R214; MPN (none) -> 0402WGF1002TCE; Manufacturer Part 0402WGF1002TCE -> (none)
- R46: renamed from R218; MPN (none) -> 0402WGF3301TCE; Manufacturer Yageo -> UNI-ROYAL(厚声); Manufacturer Part RC0402FR-073K3L -> (none); Supplier Part C137992 -> C25890
- R47: renamed from R219; MPN (none) -> 0402WGF3301TCE; Manufacturer Yageo -> UNI-ROYAL(厚声); Manufacturer Part RC0402FR-073K3L -> (none); Supplier Part C137992 -> C25890
- R48: renamed from R220; MPN (none) -> 0402WGF3301TCE; Manufacturer Yageo -> UNI-ROYAL(厚声); Manufacturer Part RC0402FR-073K3L -> (none); Supplier Part C137992 -> C25890
- R49: renamed from R221; MPN (none) -> 0402WGF3301TCE; Manufacturer Yageo -> UNI-ROYAL(厚声); Manufacturer Part RC0402FR-073K3L -> (none); Supplier Part C137992 -> C25890
- R5: renamed from R6; MPN (none) -> 0402WGF1001TCE; Manufacturer Part 0402WGF1001TCE -> (none)
- R50: renamed from R222; MPN (none) -> 0402WGF3301TCE; Manufacturer Yageo -> UNI-ROYAL(厚声); Manufacturer Part RC0402FR-073K3L -> (none); Supplier Part C137992 -> C25890
- R51: renamed from R223; MPN (none) -> 0402WGF3301TCE; Manufacturer Yageo -> UNI-ROYAL(厚声); Manufacturer Part RC0402FR-073K3L -> (none); Supplier Part C137992 -> C25890
- R52: renamed from R224; MPN (none) -> 0402WGF5101TCE; Manufacturer Part 0402WGF5101TCE -> (none)
- R53: renamed from R225; MPN (none) -> 0402WGF5101TCE; Manufacturer Part 0402WGF5101TCE -> (none)
- R54: renamed from R226; MPN (none) -> 0402WGF3300TCE; Manufacturer Part 0402WGF3300TCE -> (none)
- R55: renamed from R227; MPN (none) -> 0402WGF3300TCE; Manufacturer Part 0402WGF3300TCE -> (none)
- R56: renamed from R228; MPN (none) -> 0402WGF3300TCE; Manufacturer Part 0402WGF3300TCE -> (none)
- R57: renamed from R229; MPN (none) -> 0402WGF5101TCE; Manufacturer Part 0402WGF5101TCE -> (none)
- R58: renamed from R230; MPN (none) -> 0402WGF3300TCE; Manufacturer Part 0402WGF3300TCE -> (none)
- R6: renamed from R7; footprint MaslowMerged:R0805 -> ProPrj_Dri-easyedapro:R0402; MPN (none) -> 0402WGF1501TCE; Manufacturer Part 0805W8F1501T5E -> (none); Supplier Part C4310 -> C25867
- R7: renamed from R8; MPN (none) -> 0402WGF1001TCE; Manufacturer Part 0402WGF1001TCE -> (none)
- R8: renamed from R9; footprint MaslowMerged:R0805 -> ProPrj_Dri-easyedapro:R0402; MPN (none) -> 0402WGF5101TCE; Manufacturer Part 0805W8F5101T5E -> (none); Supplier Part C27834 -> C25905
- R9: renamed from R10; footprint MaslowMerged:R0805 -> ProPrj_Dri-easyedapro:R0402; MPN (none) -> 0402WGF1002TCE; Manufacturer Part 0805W8F1002T5E -> (none); Supplier Part C17414 -> C25744
- SW2: renamed from SW201; MPN (none) -> TSA002A3512A02; Manufacturer Part TSA002A3512A02 -> (none)
- SW3: renamed from SW202; MPN (none) -> TSA002A3512A02; Manufacturer Part TSA002A3512A02 -> (none)
- U1: MPN (none) -> XT60PB-M.G.Y; Manufacturer Part XT60PB-M.G.Y -> (none)
- U10: renamed from U201; MPN (none) -> ESP32-S3-WROOM-1-N8R2; Manufacturer Part ESP32-S3-WROOM-1-N8R2 -> (none)
- U11: renamed from U202; MPN (none) -> MP6541AGQKT-Z; Manufacturer MPS -> Monolithic Power Systems (MPS); Manufacturer Part MP6541A -> (none); Supplier Part MP6541A -> C22444490
- U12: renamed from U203; MPN (none) -> MP6541AGQKT-Z; Manufacturer MPS -> Monolithic Power Systems (MPS); Manufacturer Part MP6541A -> (none); Supplier Part MP6541A -> C22444490
- U2, U3: MPN (none) -> DRV8876PWPR; Manufacturer Part DRV8876PWPR -> (none)
- U4: renamed from U5; MPN (none) -> DRV8876PWPR; Manufacturer Part DRV8876PWPR -> (none)
- U5: renamed from U6; MPN (none) -> DRV8876PWPR; Manufacturer Part DRV8876PWPR -> (none)
- U6: renamed from U7; MPN (none) -> TCA9546APWR,118; Manufacturer Part TCA9546APWR,118 -> (none)
- U7: renamed from U9; MPN (none) -> ZDSD01GLGEAG; Manufacturer Part ZDSD01GLGEAG -> (none)
- U8: renamed from U10; MPN (none) -> ESP32-S3-WROOM-1; Manufacturer Part ESP32-S3-WROOM-1 -> (none)
- USB1: renamed from USB2; MPN (none) -> KH-TYPE-C-16P; Manufacturer Part KH-TYPE-C-16P -> (none)
- USB2: renamed from USB201; MPN (none) -> TYPE-C 16PIN; Manufacturer Part TYPE-C 16PIN -> (none)
Connections:
- net BOARDCOM1 is gone; now on net BoardCOM2: U10.32 (IO39)
- net BOARDCOM2 is gone; now on net BoardCOM1: U10.31 (IO38)
- net VIN is gone; now on net VCC: C39.1, C41.2, C43.2, C46.2, C48.2, C50.2, C53.2, C55.2, C60.1, C62.2, C64.2, C65.2, C66.2, C67.2, C70.2, C71.2, CN10.2, D3.2 (K), U11.23 (VIN), U11.25 (VIN), U12.23 (VIN), U12.25 (VIN)
- net VIN_BUCK is gone; now on net VSUP: D4.1 (K)
- net 3V3: now also C33.1, R27.1
- net BR IN2: now also U8.15 (IO3); no longer U8.14 (IO3)
- net BST: now also C31.1, U9.1 (BST)
- net Boot: now also SW1.1
- net GND: now also U8.40 (GND), U8.41 (EPAD), USB2.13 (SHELL), USB2.14 (SHELL), C28.2, C29.2, C30.2, C32.2, C33.2, R29.2, R30.2, SW1.2, U9.7 (GND), U9.9 (EP); no longer U8.39 (GND)
- net TrinamicRX: now also U8.38 (IO2); no longer U8.37 (TXD0)
- net TrinamicTX: now also U8.39 (IO1); no longer U8.37 (TXD0)
- net VSUP: now reaches D1.1 (K), D2.1 (K)
- net VSUP: now also C28.1, C32.1, U9.2 (VIN), U9.3 (EN)
- net SW_NODE: now reaches L1.1
- net SW_NODE: now also C31.2, U9.8 (SW)
- new net COMP: C30.1, R31.1, U9.6 (COMP)
- new net COMP_Z: C29.1, R31.2
- new net FB: R27.2, R29.1, U9.5 (FB)
- new net RT: R30.1, U9.4 (RT/CLK)
- no-connect marks 32 -> 31

Commit message: Before thermal vias
Parts:
- removed USB2: TYPE-C 16PIN, ProPrj_Dri-easyedapro:USB-C-SMD_TYPE-C-6PIN-2MD-073, symbol ProPrj_Dri-easyedapro:TYPE-C 16PIN 2MD(073)
- added USB2: KH-TYPE-C-16P, MaslowMerged:USB-C-SMD_KH-TYPE-C-16P, symbol KH-TYPE-C-16P
Connections:
- net CC1: now also USB2.A5 (CC1)
- net CC2: now also USB2.B5 (CC2)
- net D+: now also USB2.A6 (DP1), USB2.B6 (DP2)
- net D-: now also USB2.A7 (DN1), USB2.B7 (DN2)
- net GND: now also USB2.1 (EP), USB2.2 (EP), USB2.3 (EP), USB2.4 (EP), USB2.A1 (GND), USB2.A12 (GND), USB2.B1 (GND), USB2.B12 (GND)
- net VBUS: now also USB2.A4 (VBUS), USB2.A9 (VBUS), USB2.B4 (VBUS), USB2.B9 (VBUS)
- no-connect marks 31 -> 29
Other:
- moved on the sheet: C1, C10, C11, C12, C13, C14, C15, C16, C17, C18, C19, C2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

Commit message: Two wires left to route
Parts:
- removed R6: 1.5kΩ, ProPrj_Dri-easyedapro:R0402, symbol 0805W8F1501T5E_4
Connections:
- net TrinamicRX: no longer names the net of U8.38 (IO2)
- net TrinamicTX: no longer names the net of U8.39 (IO1)
- no-connect marks 29 -> 31
