File: Unified Control Board/Unified Control Board.kicad_sch (KiCad schematic)
At the start: 162 parts, among them CN1 B02B-PASK(LF)(SN), CN10 B3B-XH-2(LF)(SN), CN11 B3B-XH-2(LF)(SN), CN2 B02B-PASK(LF)(SN), CN3 B02B-PASK(LF)(SN), CN4 B04B-PASK(LF)(SN), CN5 B04B-PASK(LF)(SN), CN6 B02B-PASK(LF)(SN), CN7 B04B-PASK(LF)(SN), CN8 B04B-PASK(LF)(SN), CN9 B3B-XH-2(LF)(SN), Q1 ME50P06-G, SW1 TSA002A3512A02, SW2 TSA002A3512A02, SW3 TSA002A3512A02, U1 XT60PB-M.G.Y, U10 ESP32-S3-WROOM-1, U11 MP6540HA, U12 MP6540HA, U15 ADS7038QRTERQ1, U2 DRV8251ADDAR, U3 DRV8251ADDAR, U4 DRV8251ADDAR, U5 DRV8251ADDAR, U6 TCA9546A, U7 ZDSD01GLGEAG, U8 ESP32-S3-WROOM-1, U9 TPS54360BDDAR

Commit message: Replace the MP6540HA spindle drivers with the DRV8378H
The MP6540HA (5 A continuous, 6 A peak) is too small for the spindle
motors, which run 4-7 A phase peaks and reach 10-11 A under load.
U11/U12 become TI DRV8378H (23-pin VQFN-FCRLF, 6x4 mm): 65 V operating,
70 V abs max, 16 A peak, OCP fixed at 20 A, HS/LS inputs, low-side
current-sense outputs of 0.1 mA/A. It is preproduction (PDRV8378HVERR);
samples and the release date are being requested from TI.

- New MaslowMerged symbol DRV8378H and footprint VQFN-23_6x4mm_DRV8378H,
  from TI's example land pattern (SLVSH64A p.64, pad outlines taken from
  the drawing's vector data). PGND/AGND pads connect solidly to pours.
- Same nets as before: the MP6540HA support parts map across. C50/C67
  1 uF CP-to-VM, C51/C68 100 nF 100 V CPH-CPL, C52/C69 GVDD now 1 uF
  (was 4.7 uF). New C87-C94 100 nF 100 V, two per VM pin per the
  datasheet; parked right of the board edge for placement.
- SOx terminations 2.2k to 3V3 / 2.4k to GND (Rt = 1.148k): 0.115 V/A
  around 1.722 V, so -12.8 A to +13.7 A between the CSA's 0.25 V floor
  and the ADS7038's 3.3 V full scale. Rt sits just under the 1.25k where
  TI specifies +/-3% gain; calibrate the gain in firmware. LCSC codes
  for 0402WGF2201TCE/0402WGF2401TCE and the 1 uF 0805 still to fill in.

PCB: footprints swapped in place (same position and orientation), old
fan-out copper and one PHC1 trace clashing with the new pads removed.
DRC parity clean; the drivers' connections, C87-C94 placement and the
silkscreen around the larger package still need layout.

Co-Authored-By: Claude Opus 5.5 <noreply@anthropic.com>
Parts:
- removed U11, U12: MP6540HA, MaslowMerged:QFN-26_5x5mm_MP6540H, symbol MaslowMerged:MP6540HA
- added C87, C88, C89, C90, C91, C92, C93, C94: 100nF, ProPrj_Dri-easyedapro:C0603, symbol ProPrj_Dri-easyedapro:CL05B104KB54PNC
- added U11, U12: DRV8378H, MaslowMerged:VQFN-23_6x4mm_DRV8378H, symbol MaslowMerged:DRV8378H
- C52, C69: value 4.7uF/10V -> 1uF/50V; LCSC Part Name 4.7µF ±10% 16V X7R 0805 MLCC -> 1µF ±10% 50V X7R 0805 MLCC; MPN CL21A475KAQNNNE -> CL21B105KBFNNNE; Supplier Part C1779 -> LCSC: look up CL21B105KBFNNNE
- R32, R34, R36, R46, R48, R50: value 3.3kΩ -> 2.2kΩ; LCSC Part Name 3.3kΩ ±1% 1/16W 0402 Chip Resistor -> 2.2kΩ ±1% 1/16W 0402 Chip Resistor; MPN 0402WGF3301TCE -> 0402WGF2201TCE; Supplier Part C25890 -> LCSC: look up 0402WGF2201TCE
- R33, R35, R37, R47, R49, R51: value 3.3kΩ -> 2.4kΩ; LCSC Part Name 3.3kΩ ±1% 1/16W 0402 Chip Resistor -> 2.4kΩ ±1% 1/16W 0402 Chip Resistor; MPN 0402WGF3301TCE -> 0402WGF2401TCE; Supplier Part C25890 -> LCSC: look up 0402WGF2401TCE
Connections:
- net AH1: now also U11.12 (INHA)
- net AH2: now also U12.12 (INHA)
- net AL1: now also U11.9 (INLA)
- net AL2: now also U12.9 (INLA)
- net BH1: now also U11.13 (INHB)
- net BH2: now also U12.13 (INHB)
- net BL1: now also U11.10 (INLB)
- net BL2: now also U12.10 (INLB)
- net CH1: now also U11.14 (INHC)
- net CH2: now also U12.14 (INHC)
- net CL1: now also U11.11 (INLC)
- net CL2: now also U12.11 (INLC)
- net CP1_1: now also U11.1 (CPH)
- net CP1_2: now also U12.1 (CPH)
- net CP2_1: now also U11.2 (CPL)
- net CP2_2: now also U12.2 (CPL)
- net GND: now also C87.2, C88.2, C89.2, C90.2, C91.2, C92.2, C93.2, C94.2, U11.16 (PGND), U11.17 (PGND), U11.22 (AGND), U12.16 (PGND), U12.17 (PGND), U12.22 (AGND)
- net NFAULT: now also U11.8 (nFAULT)
- net NFAULT2: now also U12.8 (nFAULT)
- net NSLEEP: now also U11.15 (nSLEEP), U12.15 (nSLEEP)
- net PHA1: now also U11.7 (OUTA)
- net PHA2: now also U12.7 (OUTA)
- net PHB1: now also U11.5 (OUTB)
- net PHB2: now also U12.5 (OUTB)
- net PHC1: now also U11.3 (OUTC)
- net PHC2: now also U12.3 (OUTC)
- net SOA: now also U11.19 (SOA)
- net SOA2: now also U12.19 (SOA)
- net SOB: now also U11.20 (SOB)
- net SOB2: now also U12.20 (SOB)
- net SOC: now also U11.21 (SOC)
- net SOC2: now also U12.21 (SOC)
- net VCC: now also C87.1, C88.1, C89.1, C90.1, C91.1, C92.1, C93.1, C94.1, U11.4 (VM), U11.6 (VM), U12.4 (VM), U12.6 (VM)
- net VCP1: now also U11.23 (CP)
- net VCP2: now also U12.23 (CP)
- net VG1: now also U11.18 (GVDD)
- net VG2: now also U12.18 (GVDD)
